Commit message: add complete robot model with inertia and collision data

File: quadruped_robot_description/urdf/quadruped_robot.urdf.xacro (robot description, xacro)
@@ -1,4 +1,4 @@
 <?xml version="1.0"?>
-<robot name="quadruped_robot" xmlns:xacro="http://www.ros.org/wiki/xacro">
+<robot name="quadruped_spider" xmlns:xacro="http://www.ros.org/wiki/xacro">
     <xacro:include filename="./quadruped_robot_inertial.urdf.xacro"/>
     <!--<xacro:include filename="$(find rospackage)/path"/>-->
@@ -7,24 +7,33 @@
             <origin xyz="0 0 0.00215" rpy="0 0 0"/>
             <geometry>
-                <box size="0.074 0.074 0.0043"/>
+                <mesh filename="package://quadruped_robot_description/meshes/body_top-plate.stl"/>
             </geometry>
         </visual>
-        <collison>
+        <!--<collision>
             <origin xyz="0 0 0.00215" rpy="0 0 0" />
             <geometry>
-                <box size="0.074 0.074 0.00.0043"/>
-            </geometry>
-        </collison>
+                <box size="0.076 0.076 0.0045"/>
+            </geometry>
+        </collision>-->
+        <collision>
+            <origin xyz="0 0 0.00215" rpy="0 0 0" />
+            <geometry>
+                <mesh filename="package://quadruped_robot_description/meshes/body_top-plate_collision.stl"/>
+            </geometry>
+        </collision>
         <xacro:body_inertial/>
     </link>
+    <!-- batteries -->
+    <xacro:battery nr="1" reflect_lr="1"/>
+    <xacro:battery nr="2" reflect_lr="-1"/>
     <!-- left and right foreleg -->
     <xacro:leg leg_nr="LF" reflect_fh="1" reflect_lr="1"/>
     <xacro:leg leg_nr="RF" reflect_fh="1" reflect_lr="-1"/>
     <!-- left and right hindleg -->
-    <xacro:leg leg_nr="RH" reflect_fh="-1" reflect_lr="1"/>
-    <xacro:leg leg_nr="LH" reflect_fh="-1" reflect_lr="-1"/>
+    <xacro:leg leg_nr="LH" reflect_fh="-1" reflect_lr="1"/>
+    <xacro:leg leg_nr="RH" reflect_fh="-1" reflect_lr="-1"/>
     <xacro:macro name="leg" params="leg_nr leg_name_prefix:=Leg- reflect_fh reflect_lr">
         <xacro:property name="leg_name" value="${leg_name_prefix}${leg_nr}"/>
-        <!-- hip abduction/adduction joint -->
+        <!--###### hip abduction/adduction joint ######-->
         <joint name="${leg_name}-HAA_joint" type="revolute">
             <parent link="body_link"/><!--<parent link="${parent}"/>-->
@@ -37,19 +46,56 @@
             <!-- <calibration rising_and_or_falling=""/> -->
         </joint>
-        <!-- xacro link name here for reuse in selfCollide reference -->
-        <link name="${leg_name}-Hip_link">
-            <visual>
-                <origin xyz="0 0 0" rpy="0 0 0"/>
+        <link name="${leg_name}-Hip_link"/>
+        <joint name="${leg_name}-Hip-part1_joint" type="fixed">
+            <parent link="${leg_name}-Hip_link"/>
+            <child link="${leg_name}-Hip-part1_link"/>
+            <origin xyz="${-0.02275 + 0.012 - 0.0043/2} 0 0" rpy="0 ${-pi/2} ${pi/2 + pi/2 * reflect_fh * reflect_lr}"/>
+        </joint>
+        <link name="${leg_name}-Hip-part1_link">
+            <visual>
+                <origin xyz="0 0 0" rpy="0 0 0"/>
+                <geometry>
+                    <mesh filename="package://quadruped_robot_description/meshes/hip_part1.stl"/>
+                </geometry>
+            </visual>
+            <!--<collision>
+                <origin xyz="0 0 0" rpy="0 0 0" />
                 <geometry>
                     <box size="0.005 0.005 0.005"/>
                 </geometry>
-            </visual>
-            <collison>
+            </collision>-->
+            <collision>
+                <origin xyz="0 0 0" rpy="0 0 0" />
+                <geometry>
+                    <mesh filename="package://quadruped_robot_description/meshes/hip_part1_collision.stl"/>
+                </geometry>
+            </collision>
+            <xacro:hip_part1_inertial/>
+        </link>
+        <joint name="${leg_name}-Hip-part2_joint" type="fixed">
+            <parent link="${leg_name}-Hip_link"/>
+            <child link="${leg_name}-Hip-part2_link"/>
+            <origin xyz="0 0 0.02275" rpy="${-pi/2} ${pi/2} 0"/>
+        </joint>
+        <link name="${leg_name}-Hip-part2_link">
+            <visual>
+                <origin xyz="0 0 0" rpy="0 0 0"/>
+                <geometry>
+                    <mesh filename="package://quadruped_robot_description/meshes/hip_part2.stl"/>
+                </geometry>
+            </visual>
+            <!--<collision>
                 <origin xyz="0 0 0" rpy="0 0 0" />
                 <geometry>
                     <box size="0.005 0.005 0.005"/>
                 </geometry>
-            </collison>
-            <xacro:hip_inertial/>
+            </collision>-->
+            <collision>
+                <origin xyz="0 0 0" rpy="0 0 0" />
+                <geometry>
+                    <mesh filename="package://quadruped_robot_description/meshes/hip_part2_collision.stl"/>
+                </geometry>
+            </collision>
+            <xacro:hip_part2_inertial/>
         </link>
         <gazebo reference="${leg_name}-Hip_link">
@@ -57,13 +103,13 @@
         </gazebo>
         <xacro:servo name_suffix="${leg_name}-HAA" parent="${leg_name}-Hip_link"
-            xyz="-0.02275 0 0" rpy="${pi/2 - pi/2 * reflect_lr * reflect_fh} 0 ${pi}"/>
+            xyz="-0.02275 0 0" rpy="0 ${pi/2 + pi/2 * reflect_lr * reflect_fh} ${pi/2}"/>
         <xacro:servo name_suffix="${leg_name}-HFE" parent="${leg_name}-Hip_link"
-            xyz="0 ${-0.012  * reflect_lr * reflect_fh} 0.02275"
-            rpy="${pi/2 - pi/2 * reflect_lr * reflect_fh} 0 ${-pi/2 * reflect_lr * reflect_fh}"/>
-        <!-- hip flexion/extension joint -->
+            xyz="0 ${-(0.0077 + 0.0043/2) * reflect_lr * reflect_fh} 0.02275"
+            rpy="${pi/2 + pi/2 * reflect_lr * reflect_fh} 0 0"/>
+        <!--###### hip flexion/extension joint ######-->
         <joint name="${leg_name}-HFE_joint" type="revolute">
             <parent link="${leg_name}-Hip_link"/>
             <child link="${leg_name}-Thigh_link"/>
-            <origin xyz="0 ${-0.012 * reflect_lr * reflect_fh} 0.02275"
+            <origin xyz="0 0 0.02275"
                 rpy="${-pi/2} 0 ${-pi/2 * reflect_lr * reflect_fh}"/>
             <axis xyz="1 0 0"/>
@@ -72,17 +118,29 @@
             <!-- <calibration rising_and_or_falling=""/> -->
         </joint>
-        <link name="${leg_name}-Thigh_link">
-            <visual>
-                <origin xyz="0 0 0.0275" rpy="0 0 0"/>
-                <geometry>
-                    <box size="0.005 0.01 0.055"/>
-                </geometry>
-            </visual>
-            <collison>
-                <origin xyz="0 0 0.0275" rpy="0 0 0" />
-                <geometry>
-                    <box size="0.005 0.01 0.055"/>
-                </geometry>
-            </collison>
+        <link name="${leg_name}-Thigh_link"/>
+        <joint name="${leg_name}-Thight-part1_joint" type="fixed">
+            <parent link="${leg_name}-Thigh_link"/>
+            <child link="${leg_name}-Thigh-part1_link"/>
+            <origin xyz="${0.0077 + 0.0043} 0 0" rpy="${-pi/2} ${0} ${-pi/2}"/>
+        </joint>
+        <link name="${leg_name}-Thigh-part1_link">
+            <visual>
+                <origin xyz="0 0 0" rpy="0 0 0"/>
+                <geometry>
+                    <mesh filename="package://quadruped_robot_description/meshes/thigh.stl"/>
+                </geometry>
+            </visual>
+            <!--<collision>
+                <origin xyz="0 -0.0275 0" rpy="0 0 0" />
+                <geometry>
+                    <box size="0.02 0.075 0.0045"/>
+                </geometry>
+            </collision>-->
+            <collision>
+                <origin xyz="0 0 0" rpy="0 0 0" />
+                <geometry>
+                    <mesh filename="package://quadruped_robot_description/meshes/thigh_collision.stl"/>
+                </geometry>
+            </collision>
             <xacro:thigh_inertial/>
         </link>
@@ -90,9 +148,9 @@
             <selfCollide>true</selfCollide>
         </gazebo>
-        <!-- knee flexion/extension joint -->
+        <!--###### knee flexion/extension joint ######-->
         <joint name="${leg_name}-KFE_joint" type="revolute">
             <parent link="${leg_name}-Thigh_link"/>
             <child link="${leg_name}-Shank_link"/>
-            <origin xyz="-0.012 0 0.055" rpy="${pi/2 + pi/2 * reflect_fh * reflect_lr} 0 0"/>
+            <origin xyz="0 0 0.055" rpy="${-pi/2 * reflect_fh * reflect_lr} 0 0"/>
             <axis xyz="1 0 0"/>
             <dynamics damping="0.00001"/>
@@ -100,22 +158,34 @@
             <!-- <calibration rising_and_or_falling=""/> -->
         </joint>
-        <link name="${leg_name}-Shank_link">
-            <visual>
-                <origin xyz="0 0 0.04" rpy="0 0 0"/>
-                <geometry>
-                    <box size="0.0043 0.01 0.08"/>
-                </geometry>
-            </visual>
-            <collison>
-                <origin xyz="0 0 0.04" rpy="0 0 0" />
-                <geometry>
-                    <box size="0.0043 0.01 0.08"/>
-                </geometry>
-            </collison>
+        <link name="${leg_name}-Shank_link"/>
+        <joint name="${leg_name}-Shank_joint" type="fixed">
+            <parent link="${leg_name}-Shank_link"/>
+            <child link="${leg_name}-Shank-part1_link"/>
+            <origin xyz="0 0 0" rpy="0 ${pi/2 * reflect_fh * reflect_lr} ${pi}"/>
+        </joint>
+        <link name="${leg_name}-Shank-part1_link">
+            <visual>
+                <origin xyz="0 0 0" rpy="0 0 0"/>
+                <geometry>
+                    <mesh filename="package://quadruped_robot_description/meshes/shank.stl"/>
+                </geometry>
+            </visual>
+            <!--<collision>
+                <origin xyz="0 -0.04 0" rpy="0 0 0" />
+                <geometry>
+                    <box size="0.01 0.04 0.0045"/>
+                </geometry>
+            </collision>-->
+            <collision>
+                <origin xyz="0 0 0" rpy="0 0 0" />
+                <geometry>
+                    <mesh filename="package://quadruped_robot_description/meshes/shank_collision.stl"/>
+                </geometry>
+            </collision>
             <xacro:shank_inertial/>
         </link>
         <xacro:servo name_suffix="${leg_name}-KFE" parent="${leg_name}-Shank_link"
-            xyz="0.012 0 0"
-            rpy="${-pi/2} 0 0"/>
+            xyz="${0.0077 + 0.0043/2} 0 0"
+            rpy="0 0 ${-pi/2}"/>
         <gazebo reference="${leg_name}-Shank_link">
             <selfCollide>true</selfCollide>
@@ -128,27 +198,80 @@
             <child link="${servo_name_prefix}_link"/>
             <origin xyz="${xyz}" rpy="${rpy}"/>
-            <!--<axis xyz="1 0 0"/>
-            <dynamics damping="0.00001"/>
-            <limit lower="0.0" upper="${pi}" velocity="1.0" effort="0.0"/>-->
         </joint>
         <link name="${servo_name_prefix}_link">
             <visual>
-                <origin xyz="${-(0.0215/2 + 0.0077)} -0.007 0 " rpy="0 0 0"/>
-                <geometry>
-                    <box size="0.0215 0.024 0.012"/>
-                </geometry>
-            </visual>
-            <collison>
-                <origin xyz="${-(0.0215/2 + 0.0077)} -0.007 0 " rpy="0 0 0"/>
-                <geometry>
-                    <box size="0.0215 0.024 0.012"/>
-                </geometry>
-            </collison>
+                <origin xyz="0 0 0" rpy="0 0 0"/>
+                <geometry>
+                    <mesh filename="package://quadruped_robot_description/meshes/emax_es08a.stl"/>
+                </geometry>
+            </visual>
+            <collision>
+                <origin xyz="${-0.024/2 + 0.0058} ${-(0.0077 + 0.0043 + 0.017/2)} 0" rpy="0 0 0"/>
+                <geometry>
+                    <box size="0.024 0.017 0.012"/>
+                </geometry>
+            </collision>
             <xacro:servo_inertial/>
         </link>
-        <gazebo reference="${leg_name}-Hip_link">
+        <gazebo reference="${servo_name_prefix}_link">
             <selfCollide>true</selfCollide>
         </gazebo>
     </xacro:macro>
+    <joint name="body_bottom-plate_joint" type="fixed">"
+        <parent link="body_link"/>
+        <child link="body_bottom-plate_link"/>
+        <origin xyz="0 0 ${-(0.030 + 0.00215)}" rpy="${pi} 0 ${pi/2}"/>
+    </joint>
+    <link name="body_bottom-plate_link">
+        <visual>
+            <origin xyz="0 0 0" rpy="0 0 0"/>
+            <geometry>
+                <mesh filename="package://quadruped_robot_description/meshes/body_bottom-plate.stl"/>
+            </geometry>
+        </visual>
+        <collision>
+            <origin xyz="0 0 0.0022" rpy="0 0 0" />
+            <geometry>
+                <box size="0.076 0.076 0.0044"/>
+            </geometry>
+        </collision>
+        <xacro:body_bottom-plate_inertial/>
+    </link>
+    <xacro:macro name="battery" params="nr reflect_lr">
+        <joint name="body_battery${nr}_joint" type="fixed">"
+            <parent link="body_link"/>
+            <child link="body_battery${nr}_link"/>
+            <origin xyz="0 ${reflect_lr * 0.01} ${-(0.009 + 0.0024)}" rpy="0 ${pi/2} 0"/>
+        </joint>
+        <link name="body_battery${nr}_link">
+            <visual>
+                <origin xyz="0 0 0" rpy="0 0 0"/>
+                <geometry>
+                    <cylinder radius="0.009" length="0.065"/>
+                </geometry>
+            </visual>
+            <!--<collision>
+                <origin xyz="0 0 0" rpy="0 0 0" />
+                <geometry>
+                    <cylinder radius="0.009" length="0.065"/>
+                </geometry>
+            </collision>-->
+            <xacro:body_battery_inertial/>
+        </link>
+    </xacro:macro>
+    <joint name="body_electronic_joint" type="fixed">
+        <parent link="body_link"/>
+        <child link="body_electronic_link"/>
+        <origin xyz="0 0 ${0.0043 + 0.0081}" rpy="0 0 0"/>
+    </joint>
+    <link name="body_electronic_link">
+        <visual>
+            <origin xyz="0 0 0.001" rpy="0 0 0"/>
+            <geometry>
+                <box size="0.061 0.054 0.002"/>
+            </geometry>
+        </visual>
+        <xacro:body_electronic_inertial/>
+    </link>
     <gazebo reference="body_link">
         <selfCollide>true</selfCollide>

File: quadruped_robot_description/urdf/quadruped_robot_inertial.urdf.xacro (robot description, xacro)
@@ -1,57 +1,94 @@
 <?xml version="1.0" ?>
 <robot name="quadruped_robot" xmlns:xacro="http://ros.org/wiki/xacro">
+    <xacro:property name="densitiy_acryl" value="1.18"/> <!--g/cm^3-->
     <xacro:macro name="body_inertial">
         <inertial>
+            <origin xyz="0 0 ${0.00215 - 0.00030994730}" rpy="0 0 0"/>
+            <mass value="0.03358586"/>
+            <inertia ixx="19.14387528e-6"   ixy="0"                 ixz="0"
+                                            iyy="20.45099982e-6"    iyz="0"
+                                                                    izz="39.44674786e-6"/>
+        </inertial>
+    </xacro:macro>
+    <xacro:macro name="body_bottom-plate_inertial">
+        <inertial>
+            <origin xyz="0 0 0.00204012124" rpy="0 0 0"/>
+            <mass value="0.02916197"/>
+            <inertia ixx="13.38763183e-6"   ixy="0"                 ixz="0"
+                                            iyy="13.10624042e-6"    iyz="0"
+                                                                    izz="26.38194090e-6"/>
+        </inertial>
+    </xacro:macro>
+    <xacro:macro name="body_battery_inertial">
+        <inertial>
             <origin xyz="0 0 0" rpy="0 0 0"/>
-            <mass value="1.0"/>
+            <mass value="${0.02320757 + 0.00410292}"/>
+            <inertia ixx="${8.39147172 + 1.90379147}e-6"   ixy="0"                 ixz="0"
+                                            iyy="${8.39147160 + 1.90379147}e-6"    iyz="0"
+                                                                    izz="${0.93990666 + 0.30770938}e-6"/>
+        </inertial>
+    </xacro:macro>
+    <xacro:macro name="hip_part1_inertial">
+        <inertial>
+            <origin xyz="0.00552546327 -0.00647198504 0.0" rpy="0 0 0"/>
+            <mass value="0.00213352"/>
+            <inertia ixx="0.19721721e-6"    ixy="0.00644866e-6"     ixz="0.0"
+                                            iyy="0.12841865e-6"     iyz="0.0"
+                                                                    izz="0.31906107e-6"/>
+        </inertial>
+    </xacro:macro>
+    <xacro:macro name="hip_part2_inertial">
+        <inertial>
+            <origin xyz="0.00434707377 0.00500243858 0.0" rpy="0 0 0"/>
+            <mass value="0.00180797"/>
+            <inertia ixx="0.17081438e-6"    ixy="0.01188753e-6"     ixz="0"
+                                            iyy="0.11193880e-6"     iyz="0"
+                                                                    izz="0.27718162e-6"/>
+        </inertial>
+    </xacro:macro>
+    <xacro:macro name="thigh_inertial">
+        <inertial>
+            <origin xyz="0.0 -0.0275 0.00059547912" rpy="0 0 0"/>
+            <mass value="0.00874073"/>
+            <inertia ixx="4.10198432e-6"    ixy="0"                 ixz="0"
+                                            iyy="0.29079463e-6"     iyz="0"
+                                                                    izz="4.34650186e-6"/>
+        </inertial>
+    </xacro:macro>
+    <xacro:macro name="shank_inertial">
+        <inertial>
+            <origin xyz="-0.00228398489 -0.02353716124 0" rpy="0 0 0"/>
+            <mass value="0.00326471"/>
+            <inertia ixx="1.90216748e-6"    ixy="-0.10865983e-6"    ixz="0"
+                                            iyy="0.09630658e-6"     iyz="0"
+                                                                    izz="1.98841332e-6"/>
+        </inertial>
+    </xacro:macro>
+    <xacro:macro name="servo_inertial">
+        <inertial>
+            <origin xyz="-0.00573817801 -0.01725001328 0" rpy="0 0 0"/>
+            <mass value="0.00959970"/>
+            <inertia ixx="0.52051125e-6"    ixy="-0.05833526e-6"     ixz="-0.00000002e-6"
+                                            iyy="0.56392841e-6"      iyz="0"
+                                                                    izz="0.87703376e-6"/>
+        </inertial>
+    </xacro:macro>
+    <xacro:macro name="body_electronic_inertial">
+        <inertial>
+            <origin xyz="-0.00092815856 -0.00209563833 0.00566985182" rpy="0 0 0"/>
+            <mass value="0.039"/>
+            <inertia ixx="${6.90502970 * 1.85}e-6"  ixy="${-0.26625045 * 1.85}e-6"  ixz="${0.21982991 * 1.85}e-6"
+                                                    iyy="${5.23067546 * 1.85}e-6"   iyz="${0.51582241 * 1.85}e-6"
+                                                                                    izz="${10.47135982 * 1.85}e-6"/>
+        </inertial>
+    </xacro:macro>
+<!--<xacro:macro name="dummy_inertial">
+        <inertial>
+            <origin xyz="0 0 0" rpy="0 0 0"/>
+            <mass value="0"/>
             <inertia ixx="0"    ixy="0"     ixz="0"
                                 iyy="0"     iyz="0"
                                             izz="0"/>
         </inertial>
-    </xacro:macro>
-    <xacro:macro name="hip_inertial">
-        <inertial>
-            <origin xyz="0 0 0" rpy="0 0 0"/>
-            <mass value="1.0"/>
-            <inertia ixx="0"    ixy="0"     ixz="0"
-                                iyy="0"     iyz="0"
-                                            izz="0"/>
-        </inertial>
-    </xacro:macro>
-    <xacro:macro name="thigh_inertial">
-        <inertial>
-            <origin xyz="0 0 0" rpy="0 0 0"/>
-            <mass value="1.0"/>
-            <inertia ixx="0"    ixy="0"     ixz="0"
-                                iyy="0"     iyz="0"
-                                            izz="0"/>
-        </inertial>
-    </xacro:macro>
-    <xacro:macro name="shank_inertial">
-        <inertial>
-            <origin xyz="0 0 0" rpy="0 0 0"/>
-            <mass value="1.0"/>
-            <inertia ixx="0"    ixy="0"     ixz="0"
-                                iyy="0"     iyz="0"
-                                            izz="0"/>
-        </inertial>
-    </xacro:macro>
-    <xacro:macro name="shank_inertial">
-        <inertial>
-            <origin xyz="0 0 0" rpy="0 0 0"/>
-            <mass value="1.0"/>
-            <inertia ixx="0"    ixy="0"     ixz="0"
-                                iyy="0"     iyz="0"
-                                            izz="0"/>
-        </inertial>
-    </xacro:macro>
-    <xacro:macro name="servo_inertial">
-        <inertial>
-            <origin xyz="0 0 0" rpy="0 0 0"/>
-            <mass value="1.0"/>
-            <inertia ixx="0"    ixy="0"     ixz="0"
-                                iyy="0"     iyz="0"
-                                            izz="0"/>
-        </inertial>
-    </xacro:macro>
+    </xacro:macro>-->
 </robot>

Commit message: add dummy link which is at center of gravity for towr

File: quadruped_robot_description/urdf/quadruped_robot.urdf.xacro (robot description, xacro)
@@ -3,4 +3,10 @@
     <xacro:include filename="./quadruped_robot_inertial.urdf.xacro"/>
     <!--<xacro:include filename="$(find rospackage)/path"/>-->
+    <link name="base"/>
+    <joint name="base_joint" type="fixed">
+        <parent link="base"/>
+        <child link="body_link"/>
+        <origin xyz="0.000108 0.000244 0.006868" rpy="0 0 0"/> <!-- offset from Center of mass -->
+    </joint>
     <link name="body_link">
         <visual>
